File: PCB/PCB.kicad_pcb (KiCad board)
At the start: 2 copper layers, 6 parts, among them J3 CONN_PWR, U1 TLC5940NT

Commit message: Layout done
Parts:
- added REF**: 1pin, Connectors:1pin, F.Cu at (54.6, 137.2)
- added REF**: 1pin, Connectors:1pin, F.Cu at (121.9, 137.2)
- added REF**: 1pin, Connectors:1pin, F.Cu at (121.9, 59.7)
- added REF**: 1pin, Connectors:1pin, F.Cu at (54.6, 59.7)
Other:
- board outline added: 74.9 x 85.1 mm
Changed lines of the file:
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@@
 (kicad_pcb (version 4) (host pcbnew 4.0.6)
   (general
-    (links 63)
-    (no_connects 27)
-    (area -7.574861 -9.395 138.640001 134.6)
+    (links 0)
+    (no_connects 0)
+    (area 40.429999 54.867 138.640001 143.47)
     (thickness 1.6)
-    (drawings 0)
+    (drawings 13)
     (tracks 141)
     (zones 0)
-    (modules 6)
+    (modules 10)
     (nets 32)
   )
@@
     (pad_to_mask_clearance 0)
     (aux_axis_origin 0 0)
-    (visible_elements FFFFFF7F)
+    (visible_elements FFFFEF7F)
     (pcbplotparams
-      (layerselection 0x00030_80000001)
+      (layerselection 0x00000_00000001)
       (usegerberextensions false)
-      (excludeedgelayer true)
+      (excludeedgelayer false)
       (linewidth 0.100000)
       (plotframeref false)
@@
       (psnegative false)
       (psa4output false)
-      (plotreference true)
-      (plotvalue true)
+      (plotreference false)
+      (plotvalue false)
       (plotinvisibletext false)
       (padsonsilk false)
       (subtractmaskfromsilk false)
-      (outputformat 1)
+      (outputformat 5)
       (mirror false)
-      (drillshape 1)
+      (drillshape 0)
       (scaleselection 1)
-      (outputdirectory ""))
+      (outputdirectory ../../))
   )
   (net 0 "")
@@
     (uvia_dia 0.3)
     (uvia_drill 0.1)
-    (add_net /BLANK)
-    (add_net /GSCLK)
-    (add_net /SCLK)
-    (add_net /SIN)
-    (add_net /SOUT1)
-    (add_net /SOUT2)
-    (add_net /VCC)
-    (add_net /VLED)
-    (add_net /XLAT)
     (add_net /led-module/1DP)
     (add_net /led-module/1SEG_A)
@@
     (add_net /led-module/XLAT)
     (add_net Earth)
-    (add_net "Net-(J2-Pad1)")
-    (add_net "Net-(J2-Pad3)")
     (add_net "Net-(J_IN1-Pad10)")
     (add_net "Net-(J_IN1-Pad4)")
     (add_net "Net-(J_IN1-Pad6)")
     (add_net "Net-(J_IN1-Pad8)")
-    (add_net "Net-(J_M1-Pad10)")
-    (add_net "Net-(J_M1-Pad7)")
-    (add_net "Net-(J_M1-Pad8)")
-    (add_net "Net-(J_M1-Pad9)")
-    (add_net "Net-(J_M2-Pad10)")
-    (add_net "Net-(J_M2-Pad7)")
-    (add_net "Net-(J_M2-Pad8)")
-    (add_net "Net-(J_M2-Pad9)")
-    (add_net "Net-(J_M3-Pad10)")
-    (add_net "Net-(J_M3-Pad7)")
-    (add_net "Net-(J_M3-Pad8)")
-    (add_net "Net-(J_M3-Pad9)")
     (add_net "Net-(R1-Pad1)")
-    (add_net "Net-(SW1-Pad2)")
     (add_net "Net-(U1-Pad16)")
-    (add_net "Net-(U10-Pad1)")
-    (add_net "Net-(U10-Pad10)")
-    (add_net "Net-(U10-Pad11)")
-    (add_net "Net-(U10-Pad12)")
-    (add_net "Net-(U10-Pad14)")
-    (add_net "Net-(U10-Pad17)")
-    (add_net "Net-(U10-Pad18)")
-    (add_net "Net-(U10-Pad19)")
-    (add_net "Net-(U10-Pad2)")
-    (add_net "Net-(U10-Pad23)")
-    (add_net "Net-(U10-Pad24)")
-    (add_net "Net-(U10-Pad25)")
-    (add_net "Net-(U10-Pad26)")
-    (add_net "Net-(U10-Pad27)")
-    (add_net "Net-(U10-Pad28)")
-    (add_net "Net-(U10-Pad3)")
-    (add_net "Net-(U10-Pad4)")
-    (add_net "Net-(U10-Pad9)")
+  )
+  (module Connectors:1pin (layer F.Cu)
+    (at 54.61 137.16)
+    (descr "module 1 pin (ou trou mecanique de percage)")
+    (tags DEV)
+    (fp_text reference REF** (at 0 -3.048) (layer F.SilkS)
+      (effects (font (size 1 1) (thickness 0.15)))
+    )
+    (fp_text value 1pin (at 0 3) (layer F.Fab)
+      (effects (font (size 1 1) (thickness 0.15)))
+    )
+    (fp_circle (center 0 0) (end 2 0.8) (layer F.Fab) (width 0.1))
+    (fp_circle (center 0 0) (end 2.6 0) (layer F.CrtYd) (width 0.05))
+    (fp_circle (center 0 0) (end 0 -2.286) (layer F.SilkS) (width 0.12))
+    (pad 1 thru_hole circle (at 0 0) (size 4.064 4.064) (drill 3.048) (layers *.Cu *.Mask))
+  )
+  (module Connectors:1pin (layer F.Cu)
+    (at 121.92 137.16)
+    (descr "module 1 pin (ou trou mecanique de percage)")
+    (tags DEV)
+    (fp_text reference REF** (at 0 -3.048) (layer F.SilkS)
+      (effects (font (size 1 1) (thickness 0.15)))
+    )
+    (fp_text value 1pin (at 0 3) (layer F.Fab)
+      (effects (font (size 1 1) (thickness 0.15)))
+    )
+    (fp_circle (center 0 0) (end 2 0.8) (layer F.Fab) (width 0.1))
+    (fp_circle (center 0 0) (end 2.6 0) (layer F.CrtYd) (width 0.05))
+    (fp_circle (center 0 0) (end 0 -2.286) (layer F.SilkS) (width 0.12))
+    (pad 1 thru_hole circle (at 0 0) (size 4.064 4.064) (drill 3.048) (layers *.Cu *.Mask))
+  )
+  (module Connectors:1pin (layer F.Cu)
+    (at 121.92 59.69)
+    (descr "module 1 pin (ou trou mecanique de percage)")
+    (tags DEV)
+    (fp_text reference REF** (at 0 -3.048) (layer F.SilkS)
+      (effects (font (size 1 1) (thickness 0.15)))
+    )
+    (fp_text value 1pin (at 0 3) (layer F.Fab)
+      (effects (font (size 1 1) (thickness 0.15)))
+    )
+    (fp_circle (center 0 0) (end 2 0.8) (layer F.Fab) (width 0.1))
+    (fp_circle (center 0 0) (end 2.6 0) (layer F.CrtYd) (width 0.05))
+    (fp_circle (center 0 0) (end 0 -2.286) (layer F.SilkS) (width 0.12))
+    (pad 1 thru_hole circle (at 0 0) (size 4.064 4.064) (drill 3.048) (layers *.Cu *.Mask))
   )
   (module Connectors_WAGO:WAGO_734_3pin_Straight (layer B.Cu)
@@
     (descr "10 pins through hole IDC header")
     (tags "IDC header socket VASCH")
-    (fp_text reference J_IN1 (at 5.08 7.62) (layer B.SilkS)
+    (fp_text reference J_IN1 (at 4.6863 8.51662 180) (layer B.SilkS)
       (effects (font (size 1 1) (thickness 0.15)) (justify mirror))
     )
@@
     (fp_line (start 15.74 -3.78) (end -5.58 -3.78) (layer B.CrtYd) (width 0.05))
     (fp_line (start -5.58 -3.78) (end -5.58 6.32) (layer B.CrtYd) (width 0.05))
-    (fp_text user 1 (at 0.02 -1.72) (layer B.SilkS)
+    (fp_text user 1 (at 0.02 -1.72 180) (layer B.SilkS)
       (effects (font (size 1 1) (thickness 0.12)) (justify mirror))
     )
@@
     )
   )
+  (module Connectors:1pin (layer F.Cu)
+    (at 54.61 59.69)
+    (descr "module 1 pin (ou trou mecanique de percage)")
+    (tags DEV)
+    (fp_text reference REF** (at 0 -3.048) (layer F.SilkS)
+      (effects (font (size 1 1) (thickness 0.15)))
+    )
+    (fp_text value 1pin (at 0 3) (layer F.Fab)
+      (effects (font (size 1 1) (thickness 0.15)))
+    )
+    (fp_circle (center 0 0) (end 2 0.8) (layer F.Fab) (width 0.1))
+    (fp_circle (center 0 0) (end 2.6 0) (layer F.CrtYd) (width 0.05))
+    (fp_circle (center 0 0) (end 0 -2.286) (layer F.SilkS) (width 0.12))
+    (pad 1 thru_hole circle (at 0 0) (size 4.064 4.064) (drill 3.048) (layers *.Cu *.Mask))
+  )
+  (target plus (at 50.8 140.97) (size 5) (width 0.1) (layer Edge.Cuts))
+  (gr_line (start 64.77 134.62) (end 111.76 134.62) (layer Edge.Cuts) (width 0.1))
+  (gr_line (start 58.42 140.97) (end 64.77 134.62) (layer Edge.Cuts) (width 0.1))
+  (gr_line (start 50.8 140.97) (end 58.42 140.97) (layer Edge.Cuts) (width 0.1))
+  (gr_line (start 64.77 62.23) (end 111.76 62.23) (layer Edge.Cuts) (width 0.1))
+  (gr_line (start 58.42 55.88) (end 64.77 62.23) (layer Edge.Cuts) (width 0.1))
+  (gr_line (start 50.8 55.88) (end 58.42 55.88) (layer Edge.Cuts) (width 0.1))
+  (gr_line (start 50.8 140.97) (end 50.8 55.88) (layer Edge.Cuts) (width 0.1))
+  (gr_line (start 118.11 140.97) (end 111.76 134.62) (layer Edge.Cuts) (width 0.1))
+  (gr_line (start 125.73 140.97) (end 118.11 140.97) (layer Edge.Cuts) (width 0.1))
+  (gr_line (start 118.11 55.88) (end 111.76 62.23) (layer Edge.Cuts) (width 0.1))
+  (gr_line (start 125.73 55.88) (end 118.11 55.88) (layer Edge.Cuts) (width 0.1))
+  (gr_line (start 125.73 55.88) (end 125.73 140.97) (layer Edge.Cuts) (width 0.1))
   (segment (start 54.94782 91.39682) (end 56.361312 91.39682) (width 0.6) (layer F.Cu) (net 1))
   (segment (start 56.361312 91.39682) (end 64.039153 83.718979) (width 0.6) (layer F.Cu) (net 1))

Commit message: Some changes in PCB
Other:
- net class Default: clearance 1 -> 0.2
- rule trace_clearance: 1 -> 0.2
Changed lines of the file:
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@@
 (kicad_pcb (version 4) (host pcbnew 4.0.6)
   (general
-    (links 0)
+    (links 32)
     (no_connects 0)
-    (area 40.429999 54.867 138.640001 143.47)
+    (area 41.229999 55.667 137.840001 141.235)
     (thickness 1.6)
-    (drawings 13)
+    (drawings 12)
     (tracks 141)
     (zones 0)
@@
   (setup
     (last_trace_width 0.6)
-    (trace_clearance 1)
-    (zone_clearance 0.508)
+    (trace_clearance 0.2)
+    (zone_clearance 0.254)
     (zone_45_only no)
     (trace_min 0.2)
@@
     (pad_drill 0.6)
     (pad_to_mask_clearance 0)
-    (aux_axis_origin 0 0)
+    (aux_axis_origin 49.5 142.5)
+    (grid_origin 49.5 142.5)
     (visible_elements FFFFEF7F)
     (pcbplotparams
@@
       (viasonmask false)
       (mode 1)
-      (useauxorigin false)
+      (useauxorigin true)
       (hpglpennumber 1)
       (hpglpenspeed 20)
@@
       (padsonsilk false)
       (subtractmaskfromsilk false)
-      (outputformat 5)
+      (outputformat 1)
       (mirror false)
       (drillshape 0)
       (scaleselection 1)
-      (outputdirectory ../../))
+      (outputdirectory ../../../Downloads/foo/))
   )
   (net 0 "")
@@
   (net 31 "Net-(J_IN1-Pad6)")
   (net_class Default "This is the default net class."
-    (clearance 1)
+    (clearance 0.2)
     (trace_width 0.6)
     (via_dia 0.6)
@@
     (pad 1 thru_hole circle (at 0 0) (size 4.064 4.064) (drill 3.048) (layers *.Cu *.Mask))
   )
-  (target plus (at 50.8 140.97) (size 5) (width 0.1) (layer Edge.Cuts))
   (gr_line (start 64.77 134.62) (end 111.76 134.62) (layer Edge.Cuts) (width 0.1))
   (gr_line (start 58.42 140.97) (end 64.77 134.62) (layer Edge.Cuts) (width 0.1))
@@
   (segment (start 75.372386 118.48338) (end 74.430099 117.541093) (width 0.6) (layer F.Cu) (net 8))
   (segment (start 74.430099 117.541093) (end 74.430099 91.601767) (width 0.6) (layer F.Cu) (net 8))
-  (segment (start 93.266259 115.079781) (end 101.10978 107.23626) (width 0.6) (layer F.Cu) (net 9))
-  (segment (start 101.10978 107.23626) (end 101.10978 85.81898) (width 0.6) (layer F.Cu) (net 9))
-  (segment (start 86.7537 115.94338) (end 87.617299 115.079781) (width 0.6) (layer F.Cu) (net 9))
-  (segment (start 87.617299 115.079781) (end 93.266259 115.079781) (width 0.6) (layer F.Cu) (net 9))
+  (segment (start 93.266259 115.079781) (end 101.10978 107.23626) (width 0.8) (layer F.Cu) (net 9))
+  (segment (start 101.10978 107.23626) (end 101.10978 85.81898) (width 0.8) (layer F.Cu) (net 9))
+  (segment (start 86.7537 115.94338) (end 87.617299 115.079781) (width 0.8) (layer F.Cu) (net 9))
+  (segment (start 87.617299 115.079781) (end 93.266259 115.079781) (width 0.8) (layer F.Cu) (net 9))
   (segment (start 62.79642 90.2081) (end 67.18554 85.81898) (width 0.6) (layer F.Cu) (net 12))
   (segment (start 67.18554 85.81898) (end 73.16978 85.81898) (width 0.6) (layer F.Cu) (net 12))
