File: PCB/PCB.kicad_pcb (KiCad board)
At the start: 2 copper layers, 74.9 x 85.1 mm, 10 parts, among them J3 CONN_PWR, U1 TLC5940NT

Commit message: KiCad 4.0.7 update
Parts:
- added RV1: 2K, Potentiometers:Potentiometer_Triwood_RM-065, B.Cu at (89.5, 98.0)
- R1: value 2k -> 1k
- moved R1 9.75 mm to (95.5, 92.8), turned to 270 degrees
Connections:
- R1 pad 2: Earth -> Net-(R1-Pad2)
Routing:
- net Earth: track 58.8 -> 67.2 mm
- net Net-(R1-Pad2): track 0.00 -> 5.96 mm
- net Net-(R1-Pad1): track 11.8 -> 7.85 mm
Other:
- net class Default: clearance 0.2 -> 0.3; trace_width 0.6 -> 1
- rule trace_clearance: 0.2 -> 0.3
