File: PCB/PCB.sch (KiCad schematic (older format))
At the start: 7 parts, among them J2 BARREL_JACK, J4 CONN_02X04, U10 ATMEGA328-PU, U3 7805

Commit message: WIP
Parts:
- removed J4: CONN_02X04, Connectors:IDC_Header_Straight_8pins, symbol CONN_02X03
- added J_M1, J_M2, J_M3: CONN_IF, Connectors:IDC_Header_Straight_10pins, symbol CONN_02X05
- added SW1: SW_SPST, symbol SW_SPST
Connections:
- net labels added: SOUT1, SOUT2
- net labels removed: +12V
- wire segments 9 -> 10
Other:
- moved on the sheet: J2, JPWR1, JPWR2, JPWR3, U3

Commit message: Some changes in PCB
Parts:
- added JPWR4, JPWR5, JPWR6: CONN_PWR, Connectors_WAGO:WAGO_734_3pin_Straight, symbol CONN_01X03
- added J_M4, J_M5, J_M6, J_NET1: CONN_IF, Connectors:IDC_Header_Straight_10pins, symbol CONN_02X05
- added R?: 10K, symbol R
Connections:
- net labels added: CLK, CS, INT, RST, SCK, SI, SO, SOUT, WOL
- net labels removed: SOUT1, SOUT2
- wire segments 10 -> 53
Other:
- moved on the sheet: JPWR1, JPWR2, JPWR3

Commit message: KiCad 4.0.7 update
Parts:
- gave numbers to parts that had none: 1
Changed lines of the file:
@@
 Connection ~ 2250 7050
 $Comp
-L R R?
+L R R3
 U 1 1 592837B7
 P 3500 2500
-F 0 "R?" V 3580 2500 50  0000 C CNN
+F 0 "R3" V 3580 2500 50  0000 C CNN
 F 1 "10K" V 3500 2500 50  0000 C CNN
 F 2 "" V 3430 2500 50  0001 C CNN
@@
 VCC
 $Comp
-L Earth #PWR?
+L Earth #PWR07
 U 1 1 592846E1
 P 7550 1600
-F 0 "#PWR?" H 7550 1350 50  0001 C CNN
+F 0 "#PWR07" H 7550 1350 50  0001 C CNN
 F 1 "Earth" H 7550 1450 50  0001 C CNN
 F 2 "" H 7550 1600 50  0001 C CNN
@@
 VCC
 $Comp
-L Earth #PWR?
+L Earth #PWR08
 U 1 1 59285E83
 P 10500 2750
-F 0 "#PWR?" H 10500 2500 50  0001 C CNN
+F 0 "#PWR08" H 10500 2500 50  0001 C CNN
 F 1 "Earth" H 10500 2600 50  0001 C CNN
 F 2 "" H 10500 2750 50  0001 C CNN
@@
 VCC
 $Comp
-L Earth #PWR?
+L Earth #PWR09
 U 1 1 59285E93
 P 10500 3650
-F 0 "#PWR?" H 10500 3400 50  0001 C CNN
+F 0 "#PWR09" H 10500 3400 50  0001 C CNN
 F 1 "Earth" H 10500 3500 50  0001 C CNN
 F 2 "" H 10500 3650 50  0001 C CNN
@@
 VCC
 $Comp
-L Earth #PWR?
+L Earth #PWR010
 U 1 1 59285EA3
 P 10500 4650
-F 0 "#PWR?" H 10500 4400 50  0001 C CNN
+F 0 "#PWR010" H 10500 4400 50  0001 C CNN
 F 1 "Earth" H 10500 4500 50  0001 C CNN
 F 2 "" H 10500 4650 50  0001 C CNN
